File: Initial_Prototype/V1/PCB/Measurement_Device_PCB/Measurement_Device_PCB.kicad_pcb (KiCad board)
At the start: 2 copper layers, 14 parts

Commit message: PCB Update
Parts:
- added REF**: MountingHole_3.2mm_M3, MountingHole:MountingHole_3.2mm_M3, F.Cu at (95.0, 117.2)
- added REF**: MountingHole_3.2mm_M3, MountingHole:MountingHole_3.2mm_M3, F.Cu at (211.2, 43.0)
- added REF**: MountingHole_3.2mm_M3, MountingHole:MountingHole_3.2mm_M3, F.Cu at (211.2, 117.2)
- added REF**: MountingHole_3.2mm_M3, MountingHole:MountingHole_3.2mm_M3, F.Cu at (95.0, 43.0)
Other:
- board outline added: 125.3 x 83.2 mm
- board text added: "Prototype 1 2026-04-15 Tongji University Mély GALVEZ"
