File: Suit_Developement/Hardware/PCB/Central_Unit/Project/Central_Unit_PCB.brd (EAGLE design)
At the start: 60 x 110 mm, 24 parts, among them J1 S2B-PH-K-S(LF)(SN), J10 S4B-XH-A(LF)(SN), J11 S4B-XH-A(LF)(SN), J12 S4B-XH-A(LF)(SN), J13 S4B-XH-A(LF)(SN), J14 S4B-XH-A(LF)(SN), J2 S2B-PH-K-S(LF)(SN), J3 S2B-PH-K-S(LF)(SN), J4 S2B-PH-K-S(LF)(SN), J5 S2B-PH-K-S(LF)(SN)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

Commit message: Update
Routing:
- net A2: track 186.0 -> 180.8 mm
- net SDA_RH: track 47.8 -> 45.3 mm
- net SCL_RH: track 44.5 -> 42.0 mm
- net SCL_LA: track 18.9 -> 16.3 mm
- net SDA_LF: track 66.5 -> 68.6 mm
- net SDA_RA: track 35.9 -> 34.1 mm
- net SCL_RA: track 33.4 -> 31.6 mm
- net SDA_RF: track 45.9 -> 44.3 mm
- net SCL_RF: track 41.2 -> 39.6 mm
- net SDA_LA: track 17.4 -> 16.4 mm
- net SCL_LF: track 63.1 -> 64.1 mm
- net SDA_LH: track 136.6 -> 135.7 mm
- net 3.3V: track 282.8 -> 283.8 mm
- net A1: track 181.9 -> 181.2 mm
- net SCL_LH: track 133.7 -> 133.1 mm
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