File: Suit_Developement/Hardware/PCB/IMU/Project/IMU_PCB.brd (EAGLE design)
At the start: 27.5 x 38.3 mm, 23 parts, among them Q3 BSS138, U2 AP2112K-3.3, X2 32.768

Commit message: Update
Parts:
- moved C7 6.76 mm to (83.1, 56.1), turned to 0 degrees
- moved Q3 0.53 mm to (87.3, 58.5)
- moved X2 0.26 mm to (86.9, 61.9)
Routing:
- net 3.3V: track 72.0 -> 75.7 mm
- net SCL_3V: track 32.1 -> 32.6 mm
